File: Eagle Schematics and PCB/NeuroStimDuino.brd (EAGLE design)
At the start: 101.6 x 53.3 mm, 161 parts, among them IC1 DSPIC33FJ256GP506A-I_PT, IC10 OPA140AID, IC13 TPS73633DBVR, IC14 MIC3975-5.0YMM-TR, IC2 FT232RL, IC3 HCPL0531, IC4 HCPL0531, IC5 INA149AID, IC6 TSC2011IDT, IC7 OPA140AID, IC8 INA149AID, J1 22-27-2051-05, J2 47346-0001, J5 TMS-103-02-L-S, J6 TMS-103-02-L-S, J7 CON-SOCJ-2155, K1 LBB110P, Q1 MJE350, Q2 MJE340, Q3 MJE350, Q4 MJE340, Q8 MMBT3906, U1 AD826ARZ, U2 LT1991IMSPBF, U3 LT1991IMSPBF, U4 MCP41HV31-103E/ST, U5 MCP41HV31-103E/ST, U6 LTC4412HS6TRMPBF, U7 PMV48XP,215TO-236_SOT23_NEX-L, U8 PDME1-S5-D5-S, U9 MAX6018BEUR16+T

Commit message: NeuroStimDuino_v1.1 schematic and PCB files
Parts:
- added C11: 56nF, Capacitor_56nF:CAPC17595_87N_KEM
- added R28: 330E, rcl:R0603
- IC6: value TSC2011IDT -> TSC2012IST
- R11, R14, R18, R21: value 44.2K, 1/2W -> 35.7K
- moved F2 0.53 mm to (94.9, 8.53)
- moved U$3 0.36 mm to (94.9, 6.44)
Connections:
- net PWM10 renamed D10
- net PWM9 renamed D9
- new net N$28: C11.1, R24.2, R28.2
- net AGND: now also C11.2
- net GND: now also U4.9, U5.9; no longer U4.8, U5.8
- net N$19: now also R28.1; no longer R24.2
Routing:
- net N$19: track 43.4 -> 38.2 mm
- net N$28: track 0.00 -> 4.28 mm
- net AGND: track 220.8 -> 222.5 mm
- net GND: track 309.6 -> 310.7 mm
- net N$56: track 17.9 -> 17.4 mm
Other:
- board text added: "NeuroStimDuino v1.1"
- board text removed: "NeuroStimDuino v1.0"
